File: PCB/PiicoDev-microbit-adapter.sch (KiCad schematic (older format))
At the start: 15 parts, among them J1 Conn_01x40_Female, J10 Conn_01x01_Male, J2 Conn_01x04_Male, J5 Conn_01x04_Male, J6 Conn_01x01_Male, J7 Conn_01x01_Male, J8 Conn_01x01_Male, J9 Conn_01x01_Male

Commit message: v1 with premade microbit connector
Parts:
- J1: footprint CoreElectronics_Components:Conn_microbit_Horizontal_SMD -> CoreElectronics_Components:Conn_microbit_Right_Angle_SMT
Changed lines of the file:
@@
 F 0 "J1" H 1292 775 50  0000 C CNN
 F 1 "Conn_01x40_Female" H 1292 866 50  0000 C CNN
-F 2 "CoreElectronics_Components:Conn_microbit_Horizontal_SMD" H 1400 3000 50  0001 C CNN
+F 2 "CoreElectronics_Components:Conn_microbit_Right_Angle_SMT" H 1400 3000 50  0001 C CNN
 F 3 "~" H 1400 3000 50  0001 C CNN
 	1    1400 3000
