File: PCB/PiicoDev-microbit-adapter.sch (KiCad schematic (older format))
At the start: 15 parts, among them J1 Conn_01x40_Female, J10 Conn_01x01_Male, J2 Conn_01x04_Male, J5 Conn_01x04_Male, J6 Conn_01x01_Male, J7 Conn_01x01_Male, J8 Conn_01x01_Male, J9 Conn_01x01_Male

Commit message: Update artwork, bump to v11
Parts:
- added G2: LOGO_CoreElectronics_made-with-love, CoreElectronics_Artwork:CoreElectronics_logo_5mm_v2, symbol CoreElectronics_Artwork:LOGO_CoreElectronics_made-with-love
Changed lines of the file:
@@
 Sheet 1 1
 Title "PiicoDev Adapter for Micro:bit"
-Date "2021-03-31"
-Rev "v10"
+Date "2021-11-02"
+Rev "v11"
 Comp "Core Electronics"
 Comment1 "Designed by Michael Ruppe"
@@
 	2200 3900 2200 3800
 $Comp
-L CoreElectronics_Artwork:LOGO_CoreElectronics_made-with-love #G2
+L CoreElectronics_Artwork:LOGO_CoreElectronics_made-with-love G2
 U 1 1 6027A8F4
 P 10300 6250
-F 0 "#G2" H 10300 6044 60  0001 C CNN
+F 0 "G2" H 10300 6044 60  0001 C CNN
 F 1 "LOGO_CoreElectronics_made-with-love" H 10300 6456 60  0001 C CNN
-F 2 "" H 10300 6250 50  0001 C CNN
+F 2 "CoreElectronics_Artwork:CoreElectronics_logo_5mm_v2" H 10300 6250 50  0001 C CNN
 F 3 "" H 10300 6250 50  0001 C CNN
 	1    10300 6250
